File: pcb/Model-M-RP2040-USB.kicad_pcb (KiCad board)
At the start: 2 copper layers, 170 x 50 mm, 12 parts, among them J1 Leds, J2 Rows, J3 Columns, J4 USB-C, SW1 SWITCH, U2 USBLC6-2SC6

Commit message: WIP2
Parts:
- removed C10: 100n, Capacitor_SMD:C_0603_1608Metric
- added C1: 100n, Capacitor_SMD:C_0603_1608Metric_Pad1.08x0.95mm_HandSolder, F.Cu at (136.0, 55.5)
- added C2: 100n, Capacitor_SMD:C_0603_1608Metric_Pad1.08x0.95mm_HandSolder, F.Cu at (136.0, 58.0)
- added Q1: 2N7002, Package_TO_SOT_SMD:SOT-23, F.Cu at (140.7, 56.5)
- added U1: 74HC589, Package_SO:SOIC-16_3.9x9.9mm_P1.27mm, F.Cu at (138.1, 48.5)
- added U3: 74HC589, Package_SO:SOIC-16_3.9x9.9mm_P1.27mm, F.Cu at (152.4, 52.0)
- A1: footprint Prettylib:Raspberry_Pi_Pico_SMT_THT -> prettylib:Raspberry_Pi_Pico_SMT_THT
- J4: footprint Prettylib:HRO-TYPE-C-31-M-12-HandSoldering-NoSBU -> prettylib:HRO-TYPE-C-31-M-12-HandSoldering-NoSBU
- SW1: footprint Prettylib:TC-1109DE-X-X -> prettylib:TC-1109DE-X-X
- moved A1 0.61 mm to (67.2, 62.0)
Connections:
- A1 pad 1: unconnected-(A1-GPIO0-Pad1) -> /ROW1
- A1 pad 10: unconnected-(A1-GPIO7-Pad10) -> /ROW8
- A1 pad 11: unconnected-(A1-GPIO8-Pad11) -> /SPI1_RX
- A1 pad 12: unconnected-(A1-GPIO9-Pad12) -> /SPI1_CS
- A1 pad 14: unconnected-(A1-GPIO10-Pad14) -> /SPI1_SCK
- A1 pad 15: unconnected-(A1-GPIO11-Pad15) -> /SCROLL_LOCK
- A1 pad 16: unconnected-(A1-GPIO12-Pad16) -> /CAPS_LOCK
- A1 pad 17: unconnected-(A1-GPIO13-Pad17) -> /NUM_LOCK
- A1 pad 2: unconnected-(A1-GPIO1-Pad2) -> /ROW2
- A1 pad 30: unconnected-(A1-RUN-Pad30) -> /RUN
- A1 pad 4: unconnected-(A1-GPIO2-Pad4) -> /ROW3
- A1 pad 40: unconnected-(A1-VBUS-Pad40) -> VBUS
- A1 pad 5: unconnected-(A1-GPIO3-Pad5) -> /ROW4
- A1 pad 51: (no net) -> GND
- A1 pad 52: (no net) -> /USB_ESD_D-
- A1 pad 53: (no net) -> /USB_ESD_D+
- A1 pad 6: unconnected-(A1-GPIO4-Pad6) -> /ROW5
- A1 pad 7: unconnected-(A1-GPIO5-Pad7) -> /ROW6
- A1 pad 9: unconnected-(A1-GPIO6-Pad9) -> /ROW7
- SW1 pad 1: unconnected-(SW1-Pad1) -> GND
- SW1 pad 2: unconnected-(SW1-Pad2) -> /RUN
- U2 pad 4: /USB_D+ -> /USB_ESD_D+
- U2 pad 6: /USB_D- -> /USB_ESD_D-
Routing:
- net /USB_ESD_D+: track 0.00 -> 14.4 mm
- net /USB_ESD_D-: track 0.00 -> 12.4 mm
- net VBUS: track 23.1 -> 24.3 mm

Commit message: Rev 0.2
Parts:
- added G***: LOGO, prettylib:QMK_PoweredBy, F.Cu at (46.8, 57.2)
- added R3: 5.1k, Resistor_SMD:R_0603_1608Metric, F.Cu at (95.7, 47.9)
- added R4: 5.1k, Resistor_SMD:R_0603_1608Metric, F.Cu at (99.0, 42.9)
- added REF**: OSHW-Symbol_8.9x8mm_SilkScreen, Symbol:OSHW-Symbol_8.9x8mm_SilkScreen, F.Cu at (67.7, 57.2)
- added RN1: R_Pack04, Resistor_SMD:R_Array_Convex_4x0603, F.Cu at (87.7, 38.1)
- added RN2: R_Pack04, Resistor_SMD:R_Array_Convex_4x0603, F.Cu at (97.7, 38.1)
- added RN3: R_Pack04, Resistor_SMD:R_Array_Convex_4x0603, F.Cu at (118.0, 38.1)
- added RN4: R_Pack04, Resistor_SMD:R_Array_Convex_4x0603, F.Cu at (107.9, 38.1)
- C1, C2: footprint Capacitor_SMD:C_0603_1608Metric_Pad1.08x0.95mm_HandSolder -> Capacitor_SMD:C_0603_1608Metric
- J2: value Rows -> Rows + Leds; footprint Connector_PinSocket_2.54mm:PinSocket_1x16_P2.54mm_Vertical -> Connector_PinSocket_2.54mm:PinSocket_1x12_P2.54mm_Vertical
- J3: footprint Connector_PinSocket_2.54mm:PinSocket_1x12_P2.54mm_Vertical -> Connector_PinSocket_2.54mm:PinSocket_1x16_P2.54mm_Vertical
- J4: moved to F.Cu
- SW1: value SWITCH -> Reset
- moved J3 57.0 mm to (83.8, 34.5)
- moved C1 56.8 mm to (80.7, 42.9), turned to -90 degrees
- moved J2 56.2 mm to (140.2, 37.1)
- moved A1 52.6 mm to (119.8, 62.9)
- moved U1 50.8 mm to (87.4, 45.2), turned to 90 degrees
- moved U3 44.3 mm to (108.6, 45.2)
- moved Q1 42.6 mm to (99.0, 47.8), turned to 90 degrees
- moved C2 37.2 mm to (102.0, 42.9), turned to -90 degrees
- moved J1 5.59 mm to (177.5, 32.5), turned to -90 degrees
- moved J4 2.11 mm to (58.1, 31.3), turned to 180 degrees
- moved R2 1.52 mm to (53.7, 39.4)
- moved U2 1.52 mm to (58.0, 41.1)
- moved R1 1.52 mm to (62.3, 39.4)
- moved SW1 0.86 mm to (49.4, 30.8)
Connections:
- A1 pad 1: /ROW1 -> /SPI0_RX
- A1 pad 10: /ROW8 -> unconnected-(A1-GPIO7-Pad10)
- A1 pad 11: /SPI1_RX -> unconnected-(A1-GPIO8-Pad11)
- A1 pad 12: /SPI1_CS -> unconnected-(A1-GPIO9-Pad12)
- A1 pad 14: /SPI1_SCK -> unconnected-(A1-GPIO10-Pad14)
- A1 pad 15: /SCROLL_LOCK -> unconnected-(A1-GPIO11-Pad15)
- A1 pad 16: /CAPS_LOCK -> unconnected-(A1-GPIO12-Pad16)
- A1 pad 17: /NUM_LOCK -> unconnected-(A1-GPIO13-Pad17)
- A1 pad 2: /ROW2 -> /SPI0_CS
- A1 pad 20: unconnected-(A1-GPIO15-Pad20) -> /SCROLL_LOCK
- A1 pad 21: unconnected-(A1-GPIO16-Pad21) -> /CAPS_LOCK
- A1 pad 22: unconnected-(A1-GPIO17-Pad22) -> /NUM_LOCK
- A1 pad 24: unconnected-(A1-GPIO18-Pad24) -> /ROW8
- A1 pad 25: unconnected-(A1-GPIO19-Pad25) -> /ROW7
- A1 pad 26: unconnected-(A1-GPIO20-Pad26) -> /ROW6
- A1 pad 27: unconnected-(A1-GPIO21-Pad27) -> /ROW5
- A1 pad 29: unconnected-(A1-GPIO22-Pad29) -> /ROW4
- A1 pad 31: unconnected-(A1-GPIO26_ADC0-Pad31) -> /ROW3
- A1 pad 32: unconnected-(A1-GPIO27_ADC1-Pad32) -> /ROW2
- A1 pad 34: unconnected-(A1-GPIO28_ADC2-Pad34) -> /ROW1
- A1 pad 4: /ROW3 -> /SPI0_SCK
- A1 pad 5: /ROW4 -> /LATCH_CLK
- A1 pad 6: /ROW5 -> unconnected-(A1-GPIO4-Pad6)
- A1 pad 7: /ROW6 -> unconnected-(A1-GPIO5-Pad7)
- A1 pad 9: /ROW7 -> unconnected-(A1-GPIO6-Pad9)
- J2 pad 10: unconnected-(J2-Pin_10-Pad10) -> +3V3
- J2 pad 11: unconnected-(J2-Pin_11-Pad11) -> /CAPS_LOCK
- J2 pad 12: unconnected-(J2-Pin_12-Pad12) -> /SCROLL_LOCK
- J2 pad 9: unconnected-(J2-Pin_9-Pad9) -> /NUM_LOCK
- Q1 pad 1: /SPI1_CS -> /SPI0_CS
- U1 pad 10: /SPI1_CS -> /SPI0_CS
- U1 pad 11: /SPI1_SCK -> /SPI0_SCK
- U1 pad 12: Net-(Q1-D) -> /LATCH_CLK
- U1 pad 9: /SPI1_RX -> /SPI0_RX
- U3 pad 10: /SPI1_CS -> /SPI0_CS
- U3 pad 11: /SPI1_SCK -> /SPI0_SCK
- U3 pad 12: Net-(Q1-D) -> /LATCH_CLK
Routing:
- net +3V3: track 0.00 -> 123.6 mm, vias 0 -> 3
- net /RUN: track 0.00 -> 116.6 mm
- net /SPI0_CS: track 0.00 -> 71.1 mm, vias 0 -> 2
- net /LATCH_CLK: track 0.00 -> 68.4 mm, vias 0 -> 2
- net VBUS: track 24.3 -> 82.5 mm, vias 0 -> 1
- net /USB_ESD_D-: track 12.4 -> 69.8 mm
- net /USB_ESD_D+: track 14.4 -> 69.8 mm
- net /SPI0_SCK: track 0.00 -> 54.6 mm
- net /SPI0_RX: track 0.00 -> 47.1 mm, vias 0 -> 2
- net /SCROLL_LOCK: track 0.00 -> 40.6 mm
- net Net-(U1-SA/SerialIn): track 0.00 -> 29.2 mm
- net Net-(Q1-D): track 0.00 -> 28.5 mm, vias 0 -> 2
- net /COL8: track 0.00 -> 23.1 mm, vias 0 -> 1
- net /NUM_LOCK: track 0.00 -> 21.3 mm
- net /COL16: track 0.00 -> 21.1 mm, vias 0 -> 1
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- added copper zone on B.Cu, net GND
- added copper zone on F.Cu, net GND
Other:
- board size 170 x 50 mm -> 170 x 51.5 mm
- board text added: "CLK"
- board text added: "IBM Model M RP2040 Controller v0.2 by Stefan Kerkmann (KarlK90)"
- board text added: "IO"
